Commit message: chore: renamed hunter_something to hunter_with_arm_something
This is so we can very clearly ensure we are not conflicting with the non arm varients code

File: src/hunter_with_arm_description/description/gazebo_ros2_control_plugin.xacro (robot description, xacro)
@@ -3,5 +3,5 @@
   <gazebo>
     <plugin filename="libgazebo_ros2_control.so" name="gazebo_ros2_control">
-      <parameters>$(find hunter_description)/config/ackermann_and_arm_controller.yaml</parameters>
+      <parameters>$(find hunter_with_arm_description)/config/ackermann_and_arm_controller.yaml</parameters>
     </plugin>
   </gazebo>

File: src/hunter_with_arm_description/description/meshes.xacro (robot description, xacro)
@@ -5,5 +5,5 @@
       <origin xyz="0 0 0" rpy="0 0 0"/>
       <geometry>
-        <mesh filename="file://$(find hunter_description)/meshes/${name}.dae" />
+        <mesh filename="file://$(find hunter_with_arm_description)/meshes/${name}.dae" />
       </geometry>
     </visual>
@@ -11,5 +11,5 @@
       <origin xyz="0 0 0" rpy="0 0 0"/>
       <geometry>
-        <mesh filename="file://$(find hunter_description)/meshes/${name}.dae" />
+        <mesh filename="file://$(find hunter_with_arm_description)/meshes/${name}.dae" />
       </geometry>
     </collision>

File: src/hunter_with_arm_description/description/ros2_control.xacro (robot description, xacro)
@@ -36,5 +36,5 @@
   <gazebo>
     <plugin filename="libgazebo_ros2_control.so" name="gazebo_ros2_control">
-      <parameters>$(find hunter_description)/config/ackermann_like_controller.yaml</parameters>
+      <parameters>$(find hunter_with_arm_description)/config/ackermann_like_controller.yaml</parameters>
     </plugin>
   </gazebo>

File: src/mobile_manipulator_pltf_description/description/mobile_manipulator_pltf.urdf.xacro (robot description, xacro)
@@ -17,8 +17,8 @@
       <xacro:if value="$(arg is_sim)">
         <xacro:if value="$(arg use_arm)">
-          <xacro:include filename="$(find hunter_description)/description/robot2.urdf.xacro"/>
+          <xacro:include filename="$(find hunter_with_arm_description)/description/robot2.urdf.xacro"/>
         </xacro:if>
         <xacro:unless value="$(arg use_arm)">
-          <xacro:include filename="$(find hunter_description)/description/robot.urdf.xacro"/>
+          <xacro:include filename="$(find hunter_with_arm_description)/description/robot.urdf.xacro"/>
         </xacro:unless>
         <xacro:property name="front_lidar_rpy" value="0 0 0"/>
@@ -26,5 +26,5 @@
       </xacro:if>
       <xacro:unless value="$(arg is_sim)">
-        <xacro:include filename="$(find hunter_description)/description/robot_core_real_hack.xacro"/>
+        <xacro:include filename="$(find hunter_with_arm_description)/description/robot_core_real_hack.xacro"/>
         <xacro:property name="front_lidar_rpy" value="-0.0174533 0 0"/>
         <xacro:property name="back_lidar_rpy" value="0 0 3.14159"/>

File: src/mobile_manipulator_pltf_description/description/mobile_manipulator_pltf_org.urdf.xacro (robot description, xacro)
@@ -4,10 +4,10 @@
    <xacro:arg name="prefix" default="" />
    <xacro:if value="$(arg is_sim)">
-      <xacro:include filename="$(find hunter_description)/description/robot.urdf.xacro"/>
+      <xacro:include filename="$(find hunter_with_arm_description)/description/robot.urdf.xacro"/>
       <xacro:property name="front_lidar_rpy" value="0 0 0"/>
       <xacro:property name="back_lidar_rpy" value="0 0 3.14159"/>
    </xacro:if>
    <xacro:unless value="$(arg is_sim)">
-      <xacro:include filename="$(find hunter_description)/description/robot_core_real_hack.xacro"/>
+      <xacro:include filename="$(find hunter_with_arm_description)/description/robot_core_real_hack.xacro"/>
       <xacro:property name="front_lidar_rpy" value="-0.0174533 0 0"/>
       <xacro:property name="back_lidar_rpy" value="0 0 3.14159"/>

File: src/mobile_manipulator_pltf_description/description/mobile_manipulator_pltf_v01.urdf.xacro (robot description, xacro)
@@ -4,10 +4,10 @@
    <xacro:arg name="prefix" default="" />
    <xacro:if value="$(arg is_sim)">
-      <xacro:include filename="$(find hunter_description)/description/robot.urdf.xacro"/>
+      <xacro:include filename="$(find hunter_with_arm_description)/description/robot.urdf.xacro"/>
       <xacro:property name="front_lidar_rpy" value="0 0 0"/>
       <xacro:property name="back_lidar_rpy" value="0 0 3.14159"/>
    </xacro:if>
    <xacro:unless value="$(arg is_sim)">
-      <xacro:include filename="$(find hunter_description)/description/robot_core_real_hack.xacro"/>
+      <xacro:include filename="$(find hunter_with_arm_description)/description/robot_core_real_hack.xacro"/>
       <xacro:property name="front_lidar_rpy" value="-0.0174533 0 0"/>
       <xacro:property name="back_lidar_rpy" value="0 0 3.14159"/>

File: src/mobile_manipulator_pltf_description/description/mobile_manipulator_pltf_v02.urdf.xacro (robot description, xacro)
@@ -7,10 +7,10 @@
   <xacro:if value="$(arg use_base)">
     <xacro:if value="$(arg is_sim)">
-      <xacro:include filename="$(find hunter_description)/description/robot.urdf.xacro"/>
+      <xacro:include filename="$(find hunter_with_arm_description)/description/robot.urdf.xacro"/>
       <xacro:property name="front_lidar_rpy" value="0 0 0"/>
       <xacro:property name="back_lidar_rpy" value="0 0 3.14159"/>
     </xacro:if>
     <xacro:unless value="$(arg is_sim)">
-      <xacro:include filename="$(find hunter_description)/description/robot_core_real_hack.xacro"/>
+      <xacro:include filename="$(find hunter_with_arm_description)/description/robot_core_real_hack.xacro"/>
       <xacro:property name="front_lidar_rpy" value="-0.0174533 0 0"/>
       <xacro:property name="back_lidar_rpy" value="0 0 3.14159"/>
