Commit message: wip

File: mobile_manipulator_pltf_description/description/camera.xacro (robot description, xacro)
@@ -65,9 +65,9 @@
             <plugin name="camera_controller" filename="libgazebo_ros_camera.so" >
                 <frame_name>camera_optical_link</frame_name>
-                <camera_name>camera_01</camera_name>
+                <camera_name>arm_camera</camera_name>
                 <topic_name>image_raw</topic_name>
-                <depth_camera_info_topic_name>camera_01/camera_info</depth_camera_info_topic_name>
-                <depth_image_topic_name>camera_01/depth/image_raw</depth_image_topic_name>
-                <point_cloud_topic_name>camera_01/points</point_cloud_topic_name>
+                <depth_camera_info_topic_name>arm_camera/camera_info</depth_camera_info_topic_name>
+                <depth_image_topic_name>arm_camera/depth/image_raw</depth_image_topic_name>
+                <point_cloud_topic_name>arm_camera/points</point_cloud_topic_name>
                 <point_cloud>true</point_cloud>
             </plugin>

File: mobile_manipulator_pltf_description/description/mobile_manipulator_pltf_macro.xacro (robot description, xacro)
@@ -93,4 +93,22 @@
         <origin xyz="0 0 0" rpy="0 0 0"/>
       </xacro:robotiq_gripper>
+      <!-- Camera attached to top of the end effector -->
+      <link name="${prefix}arm_camera_link">
+        <visual>
+          <origin xyz="0 0 0" rpy="0 0 0"/>
+          <geometry>
+            <box size="0.04 0.04 0.02"/>
+          </geometry>
+          <material name="camera_gray">
+            <color rgba="0.2 0.2 0.2 1.0"/>
+          </material>
+        </visual>
+      </link>
+      <joint name="${prefix}arm_camera_joint" type="fixed">
+        <parent link="${prefix}tool0"/>
+        <child link="${prefix}arm_camera_link"/>
+        <!-- small offset above the end effector -->
+        <origin xyz="0 0 0.12" rpy="0 0 0"/>
+      </joint>
     </xacro:if>
     <!-- Disable collision between base_link_inertia (UR arm base) and chassis -->

File: mobile_manipulator_pltf_description/description/robotiq_gripper_macro.xacro (robot description, xacro)
@@ -247,5 +247,4 @@
             <origin xyz="-0.03060114 0.0 0.05490452" rpy="0 0 0" />
             <limit lower="-0.8" upper="0.0" velocity="0.5" effort="50" />
-            <mimic joint="${prefix}robotiq_85_left_knuckle_joint" multiplier="-1" />
         </joint>
         <joint name="${prefix}robotiq_85_left_finger_joint" type="fixed">
@@ -264,5 +263,4 @@
             <axis xyz="0 -1 0" />
             <origin xyz="0.0127 0.0 0.06142" rpy="0 0 0" />
-            <mimic joint="${prefix}robotiq_85_left_knuckle_joint" />
         </joint>
         <joint name="${prefix}robotiq_85_right_inner_knuckle_joint" type="continuous">
@@ -271,5 +269,4 @@
             <axis xyz="0 -1 0" />
             <origin xyz="-0.0127 0.0 0.06142" rpy="0 0 0" />
-            <mimic joint="${prefix}robotiq_85_left_knuckle_joint" multiplier="-1" />
         </joint>
         <joint name="${prefix}robotiq_85_left_finger_tip_joint" type="continuous">
@@ -278,5 +275,4 @@
             <axis xyz="0 -1 0" />
             <origin xyz="0.00563134 0.0 0.04718515" rpy="0 0 0" />
-            <mimic joint="${prefix}robotiq_85_left_knuckle_joint" multiplier="-1" />
         </joint>
         <joint name="${prefix}robotiq_85_right_finger_tip_joint" type="continuous">
@@ -285,6 +281,63 @@
             <axis xyz="0 -1 0" />
             <origin xyz="-0.00563134 0.0 0.04718515" rpy="0 0 0" />
-            <mimic joint="${prefix}robotiq_85_left_knuckle_joint" />
-        </joint>
+        </joint>
+        <!-- Gazebo-specific mimic joint plugins for Gazebo Classic simulation -->
+        <xacro:if value="${sim_gazebo}">
+            <!-- Right knuckle mimics left knuckle with multiplier -1 -->
+            <gazebo reference="${prefix}robotiq_85_right_knuckle_joint">
+                <plugin filename="libgazebo_mimic_joint_plugin.so" name="${prefix}mimic_robotiq_85_right_knuckle">
+                    <joint>${prefix}robotiq_85_right_knuckle_joint</joint>
+                    <mimicJoint>${prefix}robotiq_85_left_knuckle_joint</mimicJoint>
+                    <multiplier>-1.0</multiplier>
+                    <offset>0.0</offset>
+                    <sensitiveness>0.0</sensitiveness>
+                    <maxEffort>50.0</maxEffort>
+                </plugin>
+            </gazebo>
+            <!-- Left inner knuckle mimics left knuckle with multiplier 1 -->
+            <gazebo reference="${prefix}robotiq_85_left_inner_knuckle_joint">
+                <plugin filename="libgazebo_mimic_joint_plugin.so" name="${prefix}mimic_robotiq_85_left_inner_knuckle">
+                    <joint>${prefix}robotiq_85_left_inner_knuckle_joint</joint>
+                    <mimicJoint>${prefix}robotiq_85_left_knuckle_joint</mimicJoint>
+                    <multiplier>1.0</multiplier>
+                    <offset>0.0</offset>
+                    <sensitiveness>0.0</sensitiveness>
+                    <maxEffort>50.0</maxEffort>
+                </plugin>
+            </gazebo>
+            <!-- Right inner knuckle mimics left knuckle with multiplier -1 -->
+            <gazebo reference="${prefix}robotiq_85_right_inner_knuckle_joint">
+                <plugin filename="libgazebo_mimic_joint_plugin.so" name="${prefix}mimic_robotiq_85_right_inner_knuckle">
+                    <joint>${prefix}robotiq_85_right_inner_knuckle_joint</joint>
+                    <mimicJoint>${prefix}robotiq_85_left_knuckle_joint</mimicJoint>
+                    <multiplier>-1.0</multiplier>
+                    <offset>0.0</offset>
+                    <sensitiveness>0.0</sensitiveness>
+                    <maxEffort>50.0</maxEffort>
+                </plugin>
+            </gazebo>
+            <!-- Left finger tip mimics left knuckle with multiplier -1 -->
+            <gazebo reference="${prefix}robotiq_85_left_finger_tip_joint">
+                <plugin filename="libgazebo_mimic_joint_plugin.so" name="${prefix}mimic_robotiq_85_left_finger_tip">
+                    <joint>${prefix}robotiq_85_left_finger_tip_joint</joint>
+                    <mimicJoint>${prefix}robotiq_85_left_knuckle_joint</mimicJoint>
+                    <multiplier>-1.0</multiplier>
+                    <offset>0.0</offset>
+                    <sensitiveness>0.0</sensitiveness>
+                    <maxEffort>50.0</maxEffort>
+                </plugin>
+            </gazebo>
+            <!-- Right finger tip mimics left knuckle with multiplier 1 -->
+            <gazebo reference="${prefix}robotiq_85_right_finger_tip_joint">
+                <plugin filename="libgazebo_mimic_joint_plugin.so" name="${prefix}mimic_robotiq_85_right_finger_tip">
+                    <joint>${prefix}robotiq_85_right_finger_tip_joint</joint>
+                    <mimicJoint>${prefix}robotiq_85_left_knuckle_joint</mimicJoint>
+                    <multiplier>1.0</multiplier>
+                    <offset>0.0</offset>
+                    <sensitiveness>0.0</sensitiveness>
+                    <maxEffort>50.0</maxEffort>
+                </plugin>
+            </gazebo>
+        </xacro:if>
     </xacro:macro>
 </robot>

File: mobile_manipulator_pltf_description/description/ur5.ros2_control.xacro (robot description, xacro)
@@ -30,5 +30,5 @@
           <plugin>ign_ros2_control/IgnitionSystem</plugin>
         </xacro:if>
-        <xacro:if value="${use_fake_hardware}">
+        <xacro:if value="${use_fake_hardware and not sim_gazebo}">
           <plugin>mock_components/GenericSystem</plugin>
           <param name="fake_sensor_commands">${fake_sensor_commands}</param>
